File: TeslaCoil.kicad_pcb (KiCad board)
At the start: 2 copper layers, 29 parts, among them J1 Conn_01x03_Pin, J2 Conn_02x02_Counter_Clockwise, J3 Conn_01x03_Pin, T1 Transformer_1P_1S, U4 7815L, U5 78L05Z

Commit message: TeslaCoild pcb progress
Parts:
- D3, D4: footprint Diode_THT:Diode_Bridge_DIP-4_W7.62mm_P5.08mm -> Diode_SMD:Diode_Bridge_Vishay_DFS
- Q1, Q2: footprint Package_TO_SOT_THT:TO-220-3_Vertical -> TeslaCoil_JDG:STGB19NC60KDT4
- moved F1 71.3 mm to (122.2, 60.2), turned to 180 degrees
- moved R3 59.9 mm to (134.0, 69.2), turned to 0 degrees
- moved D4 59.3 mm to (130.3, 61.4), turned to 90 degrees
- moved C5 56.5 mm to (106.7, 117.7), turned to 0 degrees
- moved C6 56.3 mm to (98.7, 117.8), turned to 0 degrees
- moved D3 55.4 mm to (88.1, 104.9), turned to 90 degrees
- moved C9 53.3 mm to (93.6, 114.2), turned to -90 degrees
- moved C8 46.3 mm to (133.0, 75.5), turned to 0 degrees
- moved U4 40.2 mm to (101.0, 111.9), turned to 180 degrees
- moved Q1 37.1 mm to (129.4, 87.9)
- moved R2 36.6 mm to (122.4, 69.2), turned to 0 degrees
- moved C7 34.8 mm to (121.7, 75.3)
- moved U5 29.1 mm to (101.5, 103.9)
- moved Q2 22.2 mm to (128.9, 101.8)
- moved C3 21.9 mm to (112.7, 119.9), turned to 0 degrees
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Routing:
- net Net-(T1-SB): track 0.00 -> 41.5 mm
- net Net-(T1-SA): track 0.00 -> 29.5 mm
- net ANT: track 14.1 -> 38.5 mm
- net Net-(J2-Pin_1): track 7.60 -> 2.63 mm
- net Net-(U2-OUT): track 12.5 -> 17.4 mm
- net Net-(U1-2Y): track 6.92 -> 10.2 mm
- net Net-(U3-OUTA): track 5.58 -> 7.65 mm
- net Net-(J2-Pin_3): track 5.03 -> 3.29 mm
- net Net-(J2-Pin_2): track 5.68 -> 4.23 mm
- net Net-(U3-OUTB): track 4.60 -> 3.43 mm
- net GND: vias 0 -> 5
- added copper zone on F.Cu, net +15V
- added copper zone on F.Cu, net +5V
- added copper zone on B.Cu, net GND
- added copper zone on F.Cu, net GND
- added copper zone on F.Cu, net HOT
- added copper zone on F.Cu, net NTRL
- added copper zone on F.Cu, net Net-(D4-+)
- added copper zone on F.Cu, net Net-(D4--)
- added copper zone on F.Cu, net Net-(D4-Pad4)
- added copper zone on F.Cu, net Net-(J3-Pin_1)
- added copper zone on F.Cu, net Net-(J3-Pin_3)
- added copper zone on F.Cu, net Net-(Q1-Pad1)
- added copper zone on F.Cu, net Net-(Q2-Pad1)
- added copper zone on F.Cu, net VOUT

Commit message: Final PCB
Parts:
- J1: footprint Connector_PinHeader_2.54mm:PinHeader_1x03_P2.54mm_Horizontal -> Connector_Wire:SolderWire-0.5sqmm_1x03_P4.6mm_D0.9mm_OD2.1mm_Relief
- moved J1 4.61 mm to (88.0, 73.5), turned to -90 degrees
- moved U2 0.98 mm to (127.4, 115.4)
Routing:
- net Net-(U3-OUTA): track 7.65 -> 8.63 mm
- net GND: vias 5 -> 7
Other:
- board outline added: 69 x 69.5 mm
