File: Interruptor/Interruptor.kicad_pcb (KiCad board)
At the start: 2 copper layers, 27.9 x 16.1 mm, 12 parts, among them J1 USB_B_Micro, J2 Conn_01x06_Pin, SW1 SW_DPDT_x2, U2 ATtiny25-20S

Commit message: BOM, and Gerber Added
Changed lines of the file:
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@@
       (plot_on_all_layers_selection 0x0000000_00000000)
       (disableapertmacros false)
-      (usegerberextensions false)
-      (usegerberattributes true)
-      (usegerberadvancedattributes true)
-      (creategerberjobfile true)
+      (usegerberextensions true)
+      (usegerberattributes false)
+      (usegerberadvancedattributes false)
+      (creategerberjobfile false)
       (dashed_line_dash_ratio 12.000000)
       (dashed_line_gap_ratio 3.000000)
@@
       (psa4output false)
       (plotreference true)
-      (plotvalue true)
+      (plotvalue false)
       (plotinvisibletext false)
       (sketchpadsonfab false)
-      (subtractmaskfromsilk false)
+      (subtractmaskfromsilk true)
       (outputformat 1)
       (mirror false)
-      (drillshape 1)
+      (drillshape 0)
       (scaleselection 1)
-      (outputdirectory "")
+      (outputdirectory "Gerbers_Interruptor/")
     )
   )
@@
     (fp_line (start 1.6 0.8) (end -1.6 0.8)
       (stroke (width 0.1) (type solid)) (layer "F.Fab"))
-    (pad "1" smd roundrect (at -1.475 0) (size 1.15 1.8) (layers "F.Cu" "F.Paste" "F.Mask") (roundrect_rratio 0.217391)
+    (pad "1" smd roundrect (at -1.475 0) (size 1.15 1.8) (layers "F.Cu" "F.Paste" "F.Mask") (roundrect_rratio 0.2173913043)
       (net 1 "+5V") (pintype "passive"))
-    (pad "2" smd roundrect (at 1.475 0) (size 1.15 1.8) (layers "F.Cu" "F.Paste" "F.Mask") (roundrect_rratio 0.217391)
+    (pad "2" smd roundrect (at 1.475 0) (size 1.15 1.8) (layers "F.Cu" "F.Paste" "F.Mask") (roundrect_rratio 0.2173913043)
       (net 2 "GND") (pintype "passive"))
     (model "${KICAD6_3DMODEL_DIR}/Capacitor_SMD.3dshapes/C_1206_3216Metric.wrl"
@@
     (pts (xy 159.35 88.45) (xy 159.35 104.55))
     (height -2.65)
-    (gr_text "16.1000 mm" (at 160.85 96.5 90) (layer "Cmts.User")
+    (gr_text "16,1000 mm" (at 160.85 96.5 90) (layer "Cmts.User")
       (effects (font (size 1 1) (thickness 0.15)))
     )
@@
     (pts (xy 159.35 88.45) (xy 131.4 88.45))
     (height 1.65)
-    (gr_text "27.9500 mm" (at 145.375 85.65) (layer "Cmts.User")
+    (gr_text "27,9500 mm" (at 145.375 85.65) (layer "Cmts.User")
       (effects (font (size 1 1) (thickness 0.15)))
     )
