File: Interruptor/Interruptor.kicad_sch (KiCad schematic)
At the start: 12 parts, among them J1 USB_B_Micro, J2 Conn_01x06_Pin, SW1 SW_DPDT_x2, U1 ATtiny25-20S

Commit message: Finished pcb for interruptor circuit
Parts:
- SW1: footprint (none) -> Interruptor:SLW-913535-2A-RA-D
- U2: footprint (none) -> Interruptor:IF-E96E
Connections:
- net GND: now also U2.2 (-); no longer U2.
- net at R2.1: now also U2.1 (+); no longer U2.
Changed lines of the file:
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@@
       (effects (font (size 1.27 1.27)))
     )
-    (property "Footprint" "" (at 112.776 82.804 0)
+    (property "Footprint" "Interruptor:SLW-913535-2A-RA-D" (at 112.776 82.804 0)
       (effects (font (size 1.27 1.27)) hide)
     )
@@
       (effects (font (size 1.27 1.27)))
     )
-    (property "Footprint" "" (at 129.4892 85.5218 0)
+    (property "Footprint" "Interruptor:IF-E96E" (at 131.318 82.55 0)
       (effects (font (size 1.27 1.27)) hide)
     )
-    (property "Datasheet" "https://www.digikey.com/en/products/detail/industrial-fiber-optics/IF-E96E/3461614" (at 129.4892 85.5218 0)
+    (property "Datasheet" "https://www.digikey.com/en/products/detail/industrial-fiber-optics/IF-E96E/3461614" (at 128.778 92.71 0)
       (effects (font (size 1.27 1.27)) hide)
     )
-    (pin "")
-    (pin "")
+    (pin "1")
+    (pin "2")
     (instances
       (project "Tesla Coil Interrupter"

Commit message: BOM, and Gerber Added
Other:
- title: (none) -> Interruptor
Changed lines of the file:
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@@
 (kicad_sch (version 20230121) (generator eeschema)
   (paper "A4")
+  (title_block
+    (title "Interruptor")
+    (date "2023-12-01")
+    (comment 1 "Juan Daniel Gonzalez Gonzalez")
+    (comment 2 "Juan Felipe Osorio Franco")
+  )
   (junction (at 107.95 107.188) (diameter 0) (color 0 0 0 0)
   )
